File: pay-ssm_sensors.sch (KiCad schematic (older format))
At the start: 26 parts, among them J5 Screw_Terminal_1x02, J6 Screw_Terminal_1x02, J7 CONN_02X03, J8 CONN_02X03, U3 BD6231F, U4 BD6231F, U5 MCP23S17, U6 LM95071, U7 MS580301BA01, U8 HIH7131

Commit message: Reverting README.md
Parts:
- C10, C11, C7, C8, C9: footprint Capacitors_SMD:C_0603 -> (none)
- D3: footprint LEDs:LED_0603 -> (none)
- J5, J6: footprint Connectors_Terminal_Blocks:TerminalBlock_Pheonix_MKDS1.5-2pol -> (none)
- J7, J8: footprint Socket_Strips:Socket_Strip_Straight_2x03_Pitch2.54mm -> (none)
- R10, R11, R12, R13, R14, R15, R16, R7, R8, R9: footprint Resistors_SMD:R_0603 -> (none)
- U3, U4: footprint Housings_SOIC:SOIC-8_3.9x4.9mm_Pitch1.27mm -> (none)
Changed lines of the file:
@@
 F 0 "R9" V 7000 2850 50  0000 L CNN
 F 1 "10K" V 7050 2950 50  0000 L CNN
-F 2 "Resistors_SMD:R_0603" H 7050 3000 50  0001 C CNN
+F 2 "" H 7050 3000 50  0001 C CNN
 F 3 "" H 7050 3000 50  0001 C CNN
 	1    7050 3000
@@
 F 0 "R11" V 7300 2950 50  0000 L CNN
 F 1 "10K" V 7250 3050 50  0000 L CNN
-F 2 "Resistors_SMD:R_0603" H 7250 3100 50  0001 C CNN
+F 2 "" H 7250 3100 50  0001 C CNN
 F 3 "" H 7250 3100 50  0001 C CNN
 	1    7250 3100
@@
 F 0 "R10" V 7000 3050 50  0000 L CNN
 F 1 "10K" V 7050 3150 50  0000 L CNN
-F 2 "Resistors_SMD:R_0603" H 7050 3200 50  0001 C CNN
+F 2 "" H 7050 3200 50  0001 C CNN
 F 3 "" H 7050 3200 50  0001 C CNN
 	1    7050 3200
@@
 F 0 "C7" V 6300 1150 50  0000 L CNN
 F 1 "100nF" V 6500 1100 50  0000 L CNN
-F 2 "Capacitors_SMD:C_0603" H 6400 1200 50  0001 C CNN
+F 2 "" H 6400 1200 50  0001 C CNN
 F 3 "" H 6400 1200 50  0001 C CNN
 	1    6400 1200
@@
 F 0 "R8" H 6980 1420 50  0000 L CNN
 F 1 "10K" H 6980 1360 50  0000 L CNN
-F 2 "Resistors_SMD:R_0603" H 6950 1400 50  0001 C CNN
+F 2 "" H 6950 1400 50  0001 C CNN
 F 3 "" H 6950 1400 50  0001 C CNN
 	1    6950 1400
@@
 F 0 "R7" H 6930 2370 50  0000 L CNN
 F 1 "10K" H 6930 2310 50  0000 L CNN
-F 2 "Resistors_SMD:R_0603" H 6900 2350 50  0001 C CNN
+F 2 "" H 6900 2350 50  0001 C CNN
 F 3 "" H 6900 2350 50  0001 C CNN
 	1    6900 2350
@@
 F 0 "R13" V 9000 1200 50  0000 L CNN
 F 1 "10K" V 9100 1250 50  0000 L CNN
-F 2 "Resistors_SMD:R_0603" H 9100 1300 50  0001 C CNN
+F 2 "" H 9100 1300 50  0001 C CNN
 F 3 "" H 9100 1300 50  0001 C CNN
 	1    9100 1300
@@
 F 0 "C8" H 8950 1550 50  0000 L CNN
 F 1 "100nF" H 8950 1450 50  0000 L CNN
-F 2 "Capacitors_SMD:C_0603" H 8900 1500 50  0001 C CNN
+F 2 "" H 8900 1500 50  0001 C CNN
 F 3 "" H 8900 1500 50  0001 C CNN
 	1    8900 1500
@@
 F 0 "C9" H 8750 2650 50  0000 L CNN
 F 1 "100nF" H 8650 2500 50  0000 L CNN
-F 2 "Capacitors_SMD:C_0603" H 8900 2600 50  0001 C CNN
+F 2 "" H 8900 2600 50  0001 C CNN
 F 3 "" H 8900 2600 50  0001 C CNN
 	1    8900 2600
@@
 F 0 "R15" H 9980 2870 50  0000 L CNN
 F 1 "10K" H 9980 2810 50  0000 L CNN
-F 2 "Resistors_SMD:R_0603" H 9950 2850 50  0001 C CNN
+F 2 "" H 9950 2850 50  0001 C CNN
 F 3 "" H 9950 2850 50  0001 C CNN
 	1    9950 2850
@@
 F 0 "R14" H 9800 2250 50  0000 L CNN
 F 1 "10K" H 9750 2350 50  0000 L CNN
-F 2 "Resistors_SMD:R_0603" H 9950 2350 50  0001 C CNN
+F 2 "" H 9950 2350 50  0001 C CNN
 F 3 "" H 9950 2350 50  0001 C CNN
 	1    9950 2350
@@
 F 0 "C11" H 9000 4000 50  0000 L CNN
 F 1 "100nF" H 8900 3900 50  0000 L CNN
-F 2 "Capacitors_SMD:C_0603" H 9150 3950 50  0001 C CNN
+F 2 "" H 9150 3950 50  0001 C CNN
 F 3 "" H 9150 3950 50  0001 C CNN
 	1    9150 3950
@@
 F 0 "C10" H 8750 3900 50  0000 L CNN
 F 1 "0.22uF" H 8600 3800 50  0000 L CNN
-F 2 "Capacitors_SMD:C_0603" H 8900 3850 50  0001 C CNN
+F 2 "" H 8900 3850 50  0001 C CNN
 F 3 "" H 8900 3850 50  0001 C CNN
 	1    8900 3850
@@
 F 0 "R16" H 10280 3670 50  0000 L CNN
 F 1 "10K" H 10280 3610 50  0000 L CNN
-F 2 "Resistors_SMD:R_0603" H 10250 3650 50  0001 C CNN
+F 2 "" H 10250 3650 50  0001 C CNN
 F 3 "" H 10250 3650 50  0001 C CNN
 	1    10250 3650
@@
 F 0 "R12" H 8030 2220 50  0000 L CNN
 F 1 "220" H 8030 2160 50  0000 L CNN
-F 2 "Resistors_SMD:R_0603" H 8000 2200 50  0001 C CNN
+F 2 "" H 8000 2200 50  0001 C CNN
 F 3 "" H 8000 2200 50  0001 C CNN
 	1    8000 2200
@@
 F 0 "D3" V 8100 2650 50  0000 C CNN
 F 1 "LED" V 8000 2450 50  0000 C CNN
-F 2 "LEDs:LED_0603" H 8000 2550 50  0001 C CNN
+F 2 "" H 8000 2550 50  0001 C CNN
 F 3 "" H 8000 2550 50  0001 C CNN
 	1    8000 2550
@@
 F 0 "J8" H 10100 5850 50  0000 C CNN
 F 1 "CONN_02X03" H 10100 5450 50  0000 C CNN
-F 2 "Socket_Strips:Socket_Strip_Straight_2x03_Pitch2.54mm" H 10100 4450 50  0001 C CNN
+F 2 "" H 10100 4450 50  0001 C CNN
 F 3 "" H 10100 4450 50  0001 C CNN
 	1    10100 5650
@@
 F 0 "J7" H 8750 5850 50  0000 C CNN
 F 1 "CONN_02X03" H 8750 5450 50  0000 C CNN
-F 2 "Socket_Strips:Socket_Strip_Straight_2x03_Pitch2.54mm" H 8750 4450 50  0001 C CNN
+F 2 "" H 8750 4450 50  0001 C CNN
 F 3 "" H 8750 4450 50  0001 C CNN
 	1    8750 5650
@@
 F 0 "U3" H 4350 5475 60  0000 C CNN
 F 1 "BD6231F" H 4350 4725 60  0000 C CNN
-F 2 "Housings_SOIC:SOIC-8_3.9x4.9mm_Pitch1.27mm" H 4100 5100 60  0001 C CNN
+F 2 "" H 4100 5100 60  0001 C CNN
 F 3 "" H 4100 5100 60  0001 C CNN
 	1    4350 5050
@@
 F 0 "U4" H 4350 6525 60  0000 C CNN
 F 1 "BD6231F" H 4350 5775 60  0000 C CNN
-F 2 "Housings_SOIC:SOIC-8_3.9x4.9mm_Pitch1.27mm" H 4100 6150 60  0001 C CNN
+F 2 "" H 4100 6150 60  0001 C CNN
 F 3 "" H 4100 6150 60  0001 C CNN
 	1    4350 6100
@@
 F 0 "J5" H 5350 5450 50  0000 C TNN
 F 1 "Screw_Terminal_1x02" V 5200 5200 50  0000 C TNN
-F 2 "Connectors_Terminal_Blocks:TerminalBlock_Pheonix_MKDS1.5-2pol" H 5350 4975 50  0001 C CNN
+F 2 "" H 5350 4975 50  0001 C CNN
 F 3 "" H 5325 5200 50  0001 C CNN
 	1    5350 5200
@@
 F 0 "J6" H 5350 6500 50  0000 C TNN
 F 1 "Screw_Terminal_1x02" V 5200 6250 50  0000 C TNN
-F 2 "Connectors_Terminal_Blocks:TerminalBlock_Pheonix_MKDS1.5-2pol" H 5350 6025 50  0001 C CNN
+F 2 "" H 5350 6025 50  0001 C CNN
 F 3 "" H 5325 6250 50  0001 C CNN
 	1    5350 6250

Commit message: Finished the PAY SSM PCB layout.
Parts:
- added D4: V_BATT_LED, LEDs:LED_0603, symbol LED
- added J5: HEATER_1, Connectors_Terminal_Blocks:TerminalBlock_Pheonix_MPT-2.54mm_2pol, symbol Screw_Terminal_1x02
- added J6: HEATER_2, Connectors_Terminal_Blocks:TerminalBlock_Pheonix_MPT-2.54mm_2pol, symbol Screw_Terminal_1x02
- added J7: SENSOR & SPI DEBUG, Socket_Strips:Socket_Strip_Straight_2x06_Pitch2.54mm, symbol CONN_02X06
- added Q1, Q2: FCD637BNZ, pay-ssm:SOT-23-6, symbol Q_NMOS_DGS
- added R19: 10K, Resistors_SMD:R_0603, symbol R_Small
- added R7, R8: 5K, Resistors_SMD:R_0603, symbol R_Small
- C10, C11, C7, C8, C9: footprint (none) -> Capacitors_SMD:C_0603
- D3: footprint (none) -> LEDs:LED_0603
- J10: renamed from J7; footprint (none) -> Socket_Strips:Socket_Strip_Straight_2x03_Pitch2.54mm
- J11: renamed from J8; footprint (none) -> Socket_Strips:Socket_Strip_Straight_2x03_Pitch2.54mm
- J8: renamed from J5; value Screw_Terminal_1x02 -> MF_1; footprint (none) -> Connectors_Terminal_Blocks:TerminalBlock_Pheonix_MPT-2.54mm_2pol
- J9: renamed from J6; value Screw_Terminal_1x02 -> MF_2; footprint (none) -> Connectors_Terminal_Blocks:TerminalBlock_Pheonix_MPT-2.54mm_2pol
- R10: renamed from R8; footprint (none) -> Resistors_SMD:R_0603
- R11: renamed from R9; footprint (none) -> Resistors_SMD:R_0603
- R12: renamed from R10; footprint (none) -> Resistors_SMD:R_0603
- R13: renamed from R11; footprint (none) -> Resistors_SMD:R_0603
- R14: renamed from R12; footprint (none) -> Resistors_SMD:R_0603
- R15: renamed from R13; footprint (none) -> Resistors_SMD:R_0603
- R16: renamed from R14; footprint (none) -> Resistors_SMD:R_0603
- R17: renamed from R15; footprint (none) -> Resistors_SMD:R_0603
- R18: renamed from R16; footprint (none) -> Resistors_SMD:R_0603
- R9: renamed from R7; footprint (none) -> Resistors_SMD:R_0603
- U3, U4, U8: footprint (none) -> Housings_SOIC:SOIC-8_3.9x4.9mm_Pitch1.27mm
- U5: footprint (none) -> Housings_SSOP:SSOP-28_5.3x10.2mm_Pitch0.65mm
- U6: footprint (none) -> TO_SOT_Packages_SMD:SOT-23-5
- U7: footprint (none) -> pay-ssm:MS580301BA
Connections:
- net CS_1: now also J7.10 (P10)
- net CS_2: now also J7.12 (P12)
- net GND: now also D4.1 (K), Q1.3 (S), Q2.3 (S)
- net HEATER_1: now also J7.9 (P9), R7.2
- net HEATER_2: now also J7.11 (P11), R8.2
- net HUMID_CS: now also J7.8 (P8)
- net MF_1A: now also J7.1 (P1)
- net MF_1B: now also J7.3 (P3)
- net MF_2A: now also J7.5 (P5)
- net MF_2B: now also J7.7 (P7)
- net PRES_CS: now also J7.2 (P2)
- net TEMP_CS: now also J7.4 (P4)
- net TEMP_SHUTDOWN: now also J7.6 (P6)
- net V_BATT: now also J5.2, J6.2, R19.1
- new net: Q1.2 (G), R7.1
- new net: J5.1, Q1.1 (D)
- new net: J6.1, Q2.1 (D)
- new net: Q2.2 (G), R8.1
- new net: D4.2 (A), R19.2
- no-connect marks 2 -> 5
Other:
- note added: "ASSUMED MAX V_BATT:\n12VDC, 0.5A"
- note added: "MAX 25mA SOURCE\n@ 3V3"
- note removed: "REMEMBER TO SPEC MOSFET"
- note removed: "SHOULD I USE AN N OR P TYPE MOSFET? HOW SHOULD IT BE CONNECTED?"

Commit message: Added gerber outputs.
Changed lines of the file:
@@
 encoding utf-8
 Sheet 2 2
-Title ""
+Title "Payload SSM Board"
 Date ""
-Rev ""
-Comp ""
-Comment1 ""
+Rev "2"
+Comp "University of Toronto Aerospace Team"
+Comment1 "Dylan Vogel"
 Comment2 ""
 Comment3 ""
@@
 Text HLabel 1400 1050 0    60   Input ~ 0
 3V3
-Text HLabel 1400 3000 0    60   Input ~ 0
+Text HLabel 1400 2100 0    60   Input ~ 0
 GND
 Text Label 1600 1200 0    60   ~ 0
@@
 L GND #PWR055
 U 1 1 5997DC50
-P 1600 3150
-F 0 "#PWR055" H 1600 2900 50  0001 C CNN
-F 1 "GND" H 1600 3000 50  0000 C CNN
-F 2 "" H 1600 3150 50  0001 C CNN
-F 3 "" H 1600 3150 50  0001 C CNN
-	1    1600 3150
+P 1600 2250
+F 0 "#PWR055" H 1600 2000 50  0001 C CNN
+F 1 "GND" H 1600 2100 50  0000 C CNN
+F 2 "" H 1600 2250 50  0001 C CNN
+F 3 "" H 1600 2250 50  0001 C CNN
+	1    1600 2250
 	1    0    0    -1
 $EndComp
@@
 	1400 1800 1600 1800
 Wire Wire Line
-	1400 3000 1600 3000
-Wire Wire Line
-	1600 3000 1600 3150
+	1400 2100 1600 2100
+Wire Wire Line
+	1600 2100 1600 2250
 Text Label 5550 1600 2    60   ~ 0
 PRES_CS
