File: pay_ssm.kicad_pcb (KiCad board)
At the start: 4 copper layers, 98 x 84 mm, 21 parts, among them J1 RST_JMP, J2 DEBUG CONN, J3 PROGRAMMING PORT, SW1 SW_RST, U1 SN65HVD230, U2 ATMEGA32M1-MU, Y1 8MHz

Commit message: Finished the PAY SSM PCB layout.
Parts:
- added C10: 0.22uF, Capacitors_SMD:C_0603, F.Cu at (151.5, 111.6)
- added C11: 100nF, Capacitors_SMD:C_0603, F.Cu at (141.6, 111.0)
- added C7: 100nF, Capacitors_SMD:C_0603, F.Cu at (137.9, 75.7)
- added C8: 100nF, Capacitors_SMD:C_0603, F.Cu at (151.9, 103.6)
- added C9: 100nF, Capacitors_SMD:C_0603, F.Cu at (148.8, 89.9)
- added D2: LED, LEDs:LED_0603, F.Cu at (190.0, 64.4)
- added D3: LED, LEDs:LED_0603, F.Cu at (134.0, 77.5)
- added D4: V_BATT_LED, LEDs:LED_0603, F.Cu at (111.1, 79.5)
- added J10: CONN_02X03, Socket_Strips:Socket_Strip_Straight_2x03_Pitch2.54mm, F.Cu at (106.8, 109.5)
- added J11: CONN_02X03, Socket_Strips:Socket_Strip_Straight_2x03_Pitch2.54mm, F.Cu at (106.8, 121.2)
- added J12: CONN_01X08, pay-ssm:Hirose_DF14-8P-1.25H, F.Cu at (140.7, 124.0)
- added J13: CONN_01X02, Socket_Strips:Socket_Strip_Straight_1x02_Pitch2.54mm, F.Cu at (107.2, 76.6)
- added J4: RST_JMP, Socket_Strips:Socket_Strip_Straight_2x04_Pitch2.54mm, F.Cu at (186.8, 118.0)
- added J5: HEATER_1, Connectors_Terminal_Blocks:TerminalBlock_Pheonix_MPT-2.54mm_2pol, F.Cu at (107.1, 68.2)
- added J6: HEATER_2, Connectors_Terminal_Blocks:TerminalBlock_Pheonix_MPT-2.54mm_2pol, F.Cu at (107.1, 61.5)
- added J7: SENSOR & SPI DEBUG, Socket_Strips:Socket_Strip_Straight_2x06_Pitch2.54mm, F.Cu at (130.2, 101.7)
- added J8: MF_1, Connectors_Terminal_Blocks:TerminalBlock_Pheonix_MPT-2.54mm_2pol, F.Cu at (107.7, 94.0)
- added J9: MF_2, Connectors_Terminal_Blocks:TerminalBlock_Pheonix_MPT-2.54mm_2pol, F.Cu at (107.7, 84.8)
- added Q1: FCD637BNZ, pay-ssm:SOT-23-6, F.Cu at (113.9, 70.4)
- added Q2: FCD637BNZ, pay-ssm:SOT-23-6, F.Cu at (113.8, 63.6)
- added R10: 10K, Resistors_SMD:R_0603, F.Cu at (151.0, 77.5)
- added R11: 10K, Resistors_SMD:R_0603, F.Cu at (153.8, 82.4)
- added R12: 10K, Resistors_SMD:R_0603, F.Cu at (158.1, 82.4)
- added R13: 10K, Resistors_SMD:R_0603, F.Cu at (156.0, 82.4)
- added R14: 220, Resistors_SMD:R_0603, F.Cu at (134.0, 74.3)
- added R15: 10K, Resistors_SMD:R_0603, F.Cu at (140.7, 103.6)
- added R16: 10K, Resistors_SMD:R_0603, F.Cu at (143.3, 90.9)
- added R17: 10K, Resistors_SMD:R_0603, F.Cu at (143.3, 93.5)
- added R18: 10K, Resistors_SMD:R_0603, F.Cu at (139.5, 113.3)
- added R19: 10K, Resistors_SMD:R_0603, F.Cu at (111.1, 76.1)
- added R6: 120R, Resistors_SMD:R_0603, F.Cu at (189.4, 122.4)
- added R7: 5K, Resistors_SMD:R_0603, F.Cu at (117.3, 72.6)
- added R8: 5K, Resistors_SMD:R_0603, F.Cu at (117.3, 66.0)
- added R9: 10K, Resistors_SMD:R_0603, F.Cu at (137.0, 80.4)
- added U3: BD6231F, Housings_SOIC:SOIC-8_3.9x4.9mm_Pitch1.27mm, F.Cu at (117.3, 94.6)
- added U4: BD6231F, Housings_SOIC:SOIC-8_3.9x4.9mm_Pitch1.27mm, F.Cu at (117.3, 86.6)
- added U5: MCP23S17, Housings_SSOP:SSOP-28_5.3x10.2mm_Pitch0.65mm, F.Cu at (143.7, 74.7)
- added U6: LM95071, TO_SOT_Packages_SMD:SOT-23-5, F.Cu at (147.7, 92.5)
- added U7: MS580301BA01, pay-ssm:MS580301BA, F.Cu at (144.0, 100.3)
- added U8: HIH7131, Housings_SOIC:SOIC-8_3.9x4.9mm_Pitch1.27mm, F.Cu at (146.4, 112.5)
- C4: value 0.1uF -> 22pF
- C6: value 22pF -> 0.1uF
- J1: value RST_JMP -> CONN_01X08; footprint Socket_Strips:Socket_Strip_Straight_2x04_Pitch2.54mm -> pay-ssm:Hirose_DF14-8P-1.25H
- R1: value 120R -> 10K
- R2: value 10K -> 120R
- R3: value 120R -> 220
- R4: value 120R -> 1K
- R5: value 1K -> 120R
- moved J1 66.1 mm to (121.0, 124.1)
- moved R4 53.1 mm to (171.4, 72.4), turned to 0 degrees
- moved R2 30.7 mm to (186.2, 67.8)
- moved C6 29.9 mm to (164.1, 76.1)
- moved C4 29.3 mm to (161.4, 105.3), turned to 270 degrees
- moved R1 11.0 mm to (162.2, 89.2), turned to 0 degrees
- moved C5 8.89 mm to (170.3, 105.3), turned to 90 degrees
- moved R5 8.48 mm to (169.0, 80.5), turned to 180 degrees
- moved R3 3.43 mm to (186.2, 64.4)
Connections:
- C4 pad 1: +3V3 -> GND
- C4 pad 2: GND -> Net-(C4-Pad2)
- C6 pad 1: GND -> +3V3
- C6 pad 2: Net-(C6-Pad2) -> GND
- G2 pad 5: /PAY_MOSI_A -> /MOSI_A
- G2 pad 7: /PAY_MISO_A -> /MISO_A
- G2 pad 8: /PAY_SCK_A -> /SCK_A
- J1 pad 1: /RST -> +3V3
- J1 pad 2: Net-(J1-Pad2) -> /MOSI
- J1 pad 3: /MISO_A -> /MISO
- J1 pad 4: /MISO_A_COMMON -> /SCK
- J1 pad 5: /MOSI_A -> /PEX_RST
- J1 pad 6: /MOSI_A_COMMON -> /PEX_CS
- J1 pad 7: /SCK_A -> /INT_OUT
- J1 pad 8: /SCK_A_COMMON -> GND
- J2 pad 10: Net-(J2-Pad10) -> /CAN_LPWR
- J2 pad 11: Net-(J2-Pad11) -> /PEX_SSM_RST
- J2 pad 12: Net-(J2-Pad12) -> /PEX_CS
- J2 pad 13: Net-(J2-Pad13) -> /PEX_RST
- J2 pad 14: Net-(J2-Pad14) -> /INT_OUT
- R1 pad 1: /CANH -> +3V3
- R1 pad 2: /CANL -> /RST
- R2 pad 2: /RST -> Net-(D1-Pad2)
- R3 pad 1: +3V3 -> /32M1_LED
- R3 pad 2: Net-(D1-Pad2) -> Net-(D2-Pad2)
- R4 pad 1: /XXX_RST -> GND
- R4 pad 2: Net-(J1-Pad2) -> /CAN_LPWR
- R5 pad 1: GND -> /CANH
- R5 pad 2: /CAN_LPWR -> /CANL
- U2 pad 10: Net-(C5-Pad2) -> Net-(C4-Pad2)
- U2 pad 11: Net-(C6-Pad2) -> Net-(C5-Pad2)
- U2 pad 24: Net-(U2-Pad24) -> /32M1_LED
- U2 pad 25: /PAY_RST -> Net-(U2-Pad25)
- U2 pad 26: Net-(U2-Pad26) -> /PEX_CS
- U2 pad 27: Net-(U2-Pad27) -> /PEX_SSM_RST
- U2 pad 3: Net-(U2-Pad3) -> /INT_OUT
- U2 pad 30: Net-(U2-Pad30) -> /PEX_RST
- Y1 pad 1: Net-(C5-Pad2) -> Net-(C4-Pad2)
- Y1 pad 3: Net-(C6-Pad2) -> Net-(C5-Pad2)
Routing:
- net /PEX_RST: track 0.00 -> 146.4 mm, vias 0 -> 4
- net /INT_OUT: track 0.00 -> 140.1 mm, vias 0 -> 3
- net /MISO: track 81.9 -> 217.0 mm, vias 1 -> 5
- net /PEX_CS: track 0.00 -> 134.9 mm, vias 0 -> 6
- net /SCK: track 68.8 -> 199.6 mm, vias 1 -> 3
- net /MOSI: track 80.7 -> 208.3 mm, vias 1 -> 4
- net /Sensors & SPI/CS_2: track 0.00 -> 79.9 mm
- net /Sensors & SPI/CS_1: track 0.00 -> 69.6 mm
- net /PEX_SSM_RST: track 0.00 -> 67.5 mm, vias 0 -> 2
- net /Sensors & SPI/HUMID_CS: track 0.00 -> 65.1 mm, vias 0 -> 3
- net /Sensors & SPI/MF_1B: track 0.00 -> 61.8 mm, vias 0 -> 2
- net /Sensors & SPI/MF_1A: track 0.00 -> 61.6 mm
- net /Sensors & SPI/HEATER_1: track 0.00 -> 60.9 mm, vias 0 -> 2
- net /Sensors & SPI/HEATER_2: track 0.00 -> 59.8 mm, vias 0 -> 2
- net /Sensors & SPI/MF_2A: track 0.00 -> 58.1 mm, vias 0 -> 2
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- added copper zone on VCC, net +3V3
- added copper zone on B.Cu, net /V_BATT
- added copper zone on F.Cu, net /V_BATT
- added copper zone on GND, net GND
- added copper zone on F.Cu, net Net-(J5-Pad1)
- added copper zone on F.Cu, net Net-(J6-Pad1)
Other:
- net class /V_BATT added: clearance 0.2, trace_width 1, via_dia 1.5, via_drill 1
- board text added: "CAN_LPWR"
- board text added: "CS_1"
- board text added: "CS_2"
- board text added: "HEAT_1"
- board text added: "HEAT_2"
- board text added: "HUMID"
- board text added: "INT_OUT"
- board text added: "LED PCB"
- board text added: "LED_A"
- board text added: "LED_B"
- board text added: "MAX 12V 1A IN"
- board text added: "MF_1"
- board text added: "MF_1A"
- board text added: "MF_1B"
- board text added: "MF_2"
- board text added: "MF_2A"
- board text added: "MF_2B"
- board text added: "PEX_CS"
- board text added: "PEX_RST"
- board text added: "PEX_SSM"
- board text added: "PRES"
- board text added: "SENSOR PCB"
- board text added: "SPI 1"
- board text added: "SPI 2"
- board text added: "TEMP"
- board text added: "TEMP_SHUT"
- board text added: "V_BATT"
- board text removed: "DEBUGGING"
- board text removed: "DON'T FORGET TO CONNECT R4"
- board text removed: "DON'T FORGET TO RE-READ THE NETLIST AFTER CHANGING THE SCHEMATIC."
- board text removed: "REMEMBER TO CONNECT YOUR SPI_A LINES TO THE JUMPERS ONCE YOU RENAME THEM. ALSO, DON'T FORGET TO REMOVE THE TRACE FOR XXX_RST CORRESPONDING TO YOUR BOARD THIS WILL CAUSE PROBLEMS IF YOU DON'T"

Commit message: Edited silkscreen.
Other:
- board text added: "HEATER_1"
- board text added: "HEATER_2"
Changed lines of the file:
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@@
     (area 99.924999 49.924999 198.075001 134.075001)
     (thickness 1.6)
-    (drawings 80)
+    (drawings 82)
     (tracks 993)
     (zones 0)
@@
     )
   )
+  (gr_text HEATER_2 (at 102.235 61.595 270) (layer F.SilkS)
+    (effects (font (size 1 1) (thickness 0.15)))
+  )
+  (gr_text HEATER_1 (at 102.108 70.485 270) (layer F.SilkS)
+    (effects (font (size 1 1) (thickness 0.15)))
+  )
   (gr_text "MAX 12V\n1A IN" (at 116.84 78.232) (layer F.SilkS)
     (effects (font (size 1 1) (thickness 0.15)))
   )
-  (gr_text MF_2 (at 102.235 86.36 270) (layer F.SilkS)
+  (gr_text MF_2 (at 102.489 86.36 270) (layer F.SilkS)
     (effects (font (size 1 1) (thickness 0.15)))
   )
-  (gr_text MF_1 (at 102.235 95.25 270) (layer F.SilkS)
+  (gr_text MF_1 (at 102.489 95.25 270) (layer F.SilkS)
     (effects (font (size 1 1) (thickness 0.15)))
   )
@@
     (effects (font (size 1 1) (thickness 0.15)))
   )
-  (gr_text V_BATT (at 102.87 76.2 360) (layer F.SilkS)
+  (gr_text V_BATT (at 102.87 76.2) (layer F.SilkS)
     (effects (font (size 1 1) (thickness 0.15)))
   )
@@
     (effects (font (size 1 1) (thickness 0.15)))
   )
-  (gr_text "SPI 1" (at 101.6 107.315 270) (layer F.SilkS)
+  (gr_text "SPI 1" (at 102.362 107.315 270) (layer F.SilkS)
     (effects (font (size 1 1) (thickness 0.15)))
   )
-  (gr_text "SPI 2" (at 101.6 118.745 270) (layer F.SilkS)
+  (gr_text "SPI 2" (at 102.235 118.872 270) (layer F.SilkS)
     (effects (font (size 1 1) (thickness 0.15)))
   )

Commit message: Added gerber outputs.
Other:
- board text added: "UTAT SPACE SYSTEMS Heron Mk. II : PAY_SSM_V2 Designed by Dylan Vogel"
Changed lines of the file:
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@@
     (area 99.924999 49.924999 198.075001 134.075001)
     (thickness 1.6)
-    (drawings 82)
+    (drawings 83)
     (tracks 993)
     (zones 0)
@@
     (visible_elements 7FFEFFFF)
     (pcbplotparams
-      (layerselection 0x00030_80000001)
-      (usegerberextensions false)
+      (layerselection 0x010f8_80000007)
+      (usegerberextensions true)
       (excludeedgelayer true)
       (linewidth 0.100000)
@@
       (psa4output false)
       (plotreference true)
-      (plotvalue true)
+      (plotvalue false)
       (plotinvisibletext false)
       (padsonsilk false)
@@
       (outputformat 1)
       (mirror false)
-      (drillshape 1)
+      (drillshape 0)
       (scaleselection 1)
-      (outputdirectory ""))
+      (outputdirectory _exports/))
   )
   (net 0 "")
@@
     )
   )
+  (gr_text "UTAT SPACE SYSTEMS\nHeron Mk. II : PAY_SSM_V2\nDesigned by Dylan Vogel" (at 124.714 110.871) (layer F.SilkS)
+    (effects (font (size 1 1) (thickness 0.15)))
+  )
   (gr_text HEATER_2 (at 102.235 61.595 270) (layer F.SilkS)
