File: pay_ssm.sch (KiCad schematic (older format))
At the start: 24 parts, among them J1 CONN_01X08, J2 DEBUG CONN, J3 PROGRAMMING PORT, J4 RST_JMP, SW1 SW_RST, U1 ATMEGA32M1-MU, U2 SN65HVD230, Y1 8MHz

Commit message: Finished the PAY SSM PCB layout.
Parts:
- added J12: CONN_01X08, pay-ssm:Hirose_DF14-8P-1.25H, symbol CONN_01X08
- added J13: CONN_01X02, Socket_Strips:Socket_Strip_Straight_1x02_Pitch2.54mm, symbol CONN_01X02
- J1: footprint Socket_Strips:Socket_Strip_Straight_1x08_Pitch2.54mm -> pay-ssm:Hirose_DF14-8P-1.25H
- renumbered G2 to G1, G1 to G2, U2 to U1, U1 to U2
Connections:
- net +3V3: now also J12.1 (P1)
- net CAN_LPWR: now also J2.10 (P10)
- net GND: now also J12.8 (P8), J13.2 (P2)
- net INT_OUT: now also J2.14 (P14)
- net MISO: now also J12.3 (P3)
- net MOSI: now also J12.2 (P2)
- net PAY_RST: no longer U2.25 ((PCINT15/D2A/AMP2+)PC7)
- net PEX_CS: now also J2.12 (P12), J12.6 (P6)
- net PEX_RST: now also J2.13 (P13), J12.5 (P5)
- net PEX_SSM_RST: now also J2.11 (P11)
- net SCK: now also J12.4 (P4)
- net V_BATT: now also J13.1 (P1)
- no-connect marks 5 -> 11
Other:
- note added: "I/O SENSORS"
- note added: "INCOMING HIGH VOLTAGE"
- note added: "OUTGOING LEDS"
- note removed: "OUTGOING"
Changed lines of the file:
@@
 CANH
 $Comp
-L CONN_02X10 G2
+L CONN_02X10 G1
 U 1 1 598FD923
 P 9650 2950
-F 0 "G2" H 9650 3500 50  0000 C CNN
+F 0 "G1" H 9650 3500 50  0000 C CNN
 F 1 "GENERAL CONN 1" V 9650 2950 50  0000 C CNN
 F 2 "Socket_Strips:Socket_Strip_Straight_2x10_Pitch2.54mm" H 9650 1750 50  0001 C CNN
@@
 $EndComp
 $Comp
-L CONN_02X10 G1
+L CONN_02X10 G2
 U 1 1 598FD960
 P 9650 1650
-F 0 "G1" H 9650 2200 50  0000 C CNN
+F 0 "G2" H 9650 2200 50  0000 C CNN
 F 1 "GENERAL CONN 2" V 9650 1650 50  0000 C CNN
 F 2 "Socket_Strips:Socket_Strip_Straight_2x10_Pitch2.54mm" H 9650 450 50  0001 C CNN
@@
 Text Label 4050 2850 0    60   ~ 0
 COM_RST
-Text Label 4050 2950 0    60   ~ 0
-PAY_RST
 $Comp
 L LED D1
@@
 PAY_RST
 $Comp
-L SN65HVD233 U2
+L SN65HVD233 U1
 U 1 1 599066B1
 P 6800 2050
-F 0 "U2" H 7150 2500 60  0000 R CNN
+F 0 "U1" H 7150 2500 60  0000 R CNN
 F 1 "SN65HVD230" H 6800 1600 60  0000 C CNN
-F 2 "Housings_SOIC:SOIC-8_3.9x4.9mm_Pitch1.27mm" H 6800 1525 30  0000 C CNN
+F 2 "Housings_SOIC:SOIC-8_3.9x4.9mm_Pitch1.27mm" H 6800 1525 30  0001 C CNN
 F 3 "" H 6800 2050 60  0000 C CNN
 	1    6800 2050
@@
 $EndComp
 $Comp
-L ATMEGA32M1-MU U1
+L ATMEGA32M1-MU U2
 U 1 1 59464C0C
 P 2650 3050
-F 0 "U1" H 1700 4880 50  0000 L BNN
+F 0 "U2" H 1700 4880 50  0000 L BNN
 F 1 "ATMEGA32M1-MU" H 3150 1650 50  0000 L BNN
 F 2 "Housings_QFP:TQFP-32_7x7mm_Pitch0.8mm" H 2650 3050 50  0001 C CIN
@@
 F 0 "J1" H 4200 6750 50  0000 C CNN
 F 1 "CONN_01X08" V 4300 6300 50  0000 C CNN
-F 2 "Socket_Strips:Socket_Strip_Straight_1x08_Pitch2.54mm" H 4200 6300 50  0001 C CNN
+F 2 "pay-ssm:Hirose_DF14-8P-1.25H" H 4200 6300 50  0001 C CNN
 F 3 "" H 4200 6300 50  0001 C CNN
 	1    4200 6300
 	1    0    0    -1
 $EndComp
-Text Notes 3950 7050 0    60   ~ 0
-OUTGOING
+Text Notes 3700 7100 0    60   ~ 0
+I/O SENSORS
 $Comp
 L +3V3 #PWR030
@@
 Wire Wire Line
 	4050 2850 3750 2850
-Wire Wire Line
-	4050 2950 3750 2950
 Wire Wire Line
 	3750 2650 4050 2650
@@
 Text Label 6050 4600 2    60   ~ 0
 V_BATT
+NoConn ~ 3750 2950
+Wire Wire Line
+	6050 4600 6300 4600
+Text Label 7350 5800 2    60   ~ 0
+V_BATT
+Text Label 9400 4200 2    60   ~ 0
+PEX_SSM_RST
+Text Label 9400 4300 2    60   ~ 0
+PEX_RST
+Text Label 9900 4200 0    60   ~ 0
+PEX_CS
+Text Label 9900 4300 0    60   ~ 0
+INT_OUT
+Text Label 9900 4100 0    60   ~ 0
+CAN_LPWR
+NoConn ~ 9900 4000
+NoConn ~ 9900 4400
+NoConn ~ 9400 4400
+NoConn ~ 9950 2700
+$Comp
+L CONN_01X02 J13
+U 1 1 599A077F
+P 7650 5850
+F 0 "J13" H 7650 6000 50  0000 C CNN
+F 1 "CONN_01X02" V 7750 5850 50  0000 C CNN
+F 2 "Socket_Strips:Socket_Strip_Straight_1x02_Pitch2.54mm" H 7650 5850 50  0001 C CNN
+F 3 "" H 7650 5850 50  0001 C CNN
+	1    7650 5850
+	1    0    0    -1
+$EndComp
+Wire Wire Line
+	7350 5800 7450 5800
+$Comp
+L GND #PWR034
+U 1 1 599A0AA8
+P 7400 6000
+F 0 "#PWR034" H 7400 5750 50  0001 C CNN
+F 1 "GND" H 7400 5850 50  0000 C CNN
+F 2 "" H 7400 6000 50  0001 C CNN
+F 3 "" H 7400 6000 50  0001 C CNN
+	1    7400 6000
+	1    0    0    -1
+$EndComp
+Wire Wire Line
+	7400 6000 7400 5900
+Wire Wire Line
+	7400 5900 7450 5900
+Text Notes 6850 6400 0    60   ~ 0
+INCOMING HIGH VOLTAGE
+$Comp
+L CONN_01X08 J12
+U 1 1 599A0F98
+P 5700 6300
+F 0 "J12" H 5700 6750 50  0000 C CNN
+F 1 "CONN_01X08" V 5800 6300 50  0000 C CNN
+F 2 "pay-ssm:Hirose_DF14-8P-1.25H" H 5700 6300 50  0001 C CNN
+F 3 "" H 5700 6300 50  0001 C CNN
+	1    5700 6300
+	1    0    0    -1
+$EndComp
+Text Notes 5150 7100 0    60   ~ 0
+OUTGOING LEDS
+$Comp
+L +3V3 #PWR035
+U 1 1 599A0F9F
+P 5400 5850
+F 0 "#PWR035" H 5400 5700 50  0001 C CNN
+F 1 "+3V3" H 5400 5990 50  0000 C CNN
+F 2 "" H 5400 5850 50  0001 C CNN
+F 3 "" H 5400 5850 50  0001 C CNN
+	1    5400 5850
+	1    0    0    -1
+$EndComp
+$Comp
+L GND #PWR036
+U 1 1 599A0FA5
+P 5400 6750
+F 0 "#PWR036" H 5400 6500 50  0001 C CNN
+F 1 "GND" H 5400 6600 50  0000 C CNN
+F 2 "" H 5400 6750 50  0001 C CNN
+F 3 "" H 5400 6750 50  0001 C CNN
+	1    5400 6750
+	1    0    0    -1
+$EndComp
+Text Label 5400 6050 2    60   ~ 0
+MOSI
+Text Label 5400 6150 2    60   ~ 0
+MISO
+Text Label 5400 6250 2    60   ~ 0
+SCK
+Text Label 5400 6350 2    60   ~ 0
+PEX_RST
+Text Label 5400 6450 2    60   ~ 0
+PEX_CS
+Wire Wire Line
+	5400 6750 5400 6650
+Wire Wire Line
+	5400 6650 5500 6650
+Wire Wire Line
+	5400 6550 5500 6550
+Wire Wire Line
+	5400 5850 5400 5950
+Wire Wire Line
+	5400 5950 5500 5950
+Wire Wire Line
+	5400 6050 5500 6050
+Wire Wire Line
+	5400 6150 5500 6150
+Wire Wire Line
+	5400 6250 5500 6250
+Wire Wire Line
+	5400 6350 5500 6350
+Wire Wire Line
+	5400 6450 5500 6450
+NoConn ~ 5400 6550
 $EndSCHEMATC
